File: pcb/pcb.kicad_pcb (KiCad board)
At the start: 2 copper layers, 1 part

Commit message: Schematic Donezo
Parts:
- removed REF**: RPi_Pico_SMD_TH, MCU_RPI:RPi_Pico_SMD_TH
- added C1: 10u, Capacitor_SMD:C_0603_1608Metric, F.Cu at (147.2, 66.3)
- added C2: 10u, Capacitor_SMD:C_0603_1608Metric, F.Cu at (147.2, 68.8)
- added D1: SK6812MINI, LED_SMD:LED_WS2812B_PLCC4_5.0x5.0mm_P3.2mm, F.Cu at (71.2, 129.5)
- added D2: SK6812MINI, LED_SMD:LED_WS2812B_PLCC4_5.0x5.0mm_P3.2mm, F.Cu at (137.0, 89.2)
- added D3: SK6812MINI, LED_SMD:LED_WS2812B_PLCC4_5.0x5.0mm_P3.2mm, F.Cu at (137.0, 95.8)
- added D4: SK6812MINI, LED_SMD:LED_WS2812B_PLCC4_5.0x5.0mm_P3.2mm, F.Cu at (137.0, 102.4)
- added J1: USB4085-GF-A_REVB, USB-C:GCT_USB4085-GF-A_REVB, F.Cu at (150.8, 60.0)
- added J2: AudioJack4, Connector_Audio:Jack_3.5mm_PJ320D_Horizontal, F.Cu at (195.9, 68.6)
- added J3: AudioJack4, Connector_Audio:Jack_3.5mm_PJ320D_Horizontal, F.Cu at (155.1, 95.8)
- added J6: Conn_01x08_Pin, Connector_PinHeader_2.54mm:PinHeader_1x08_P2.54mm_Vertical, F.Cu at (143.5, 81.6)
- added R2: 5k1, Capacitor_SMD:C_0603_1608Metric, F.Cu at (147.2, 71.3)
- added R3: 5k1, Capacitor_SMD:C_0603_1608Metric, F.Cu at (147.2, 73.8)
- added SW1: SW_Push, Button_Switch_Keyboard:SW_Cherry_MX_1.00u_PCB, F.Cu at (63.7, 114.4)
- added SW2: SW_Push, Button_Switch_Keyboard:SW_Cherry_MX_1.00u_PCB, F.Cu at (63.7, 134.6)
- added SW3: SW_Push, Button_Switch_Keyboard:SW_Cherry_MX_1.00u_PCB, F.Cu at (83.9, 114.4)
- added SW4: SW_Push, Button_Switch_Keyboard:SW_Cherry_MX_1.00u_PCB, F.Cu at (83.9, 134.6)
- added SW5: SW_Push, Button_Switch_Keyboard:SW_Cherry_MX_1.00u_PCB, F.Cu at (104.1, 114.4)
- added SW6: SW_Push, Button_Switch_Keyboard:SW_Cherry_MX_1.00u_PCB, F.Cu at (104.1, 134.6)
- added SW7: RotaryEncoder_Switch, Rotary_Encoder:RotaryEncoder_Alps_EC11E-Switch_Vertical_H20mm, F.Cu at (33.4, 137.2)
- added SW8: RotaryEncoder_Switch, Rotary_Encoder:RotaryEncoder_Alps_EC11E_Vertical_H20mm, F.Cu at (33.5, 116.9)
- added U1: Pico, Library:RPi_Pico_SMD_TH, F.Cu at (66.0, 95.2)
- added U2: Pico, Library:RPi_Pico_SMD_TH, F.Cu at (222.2, 100.3)
- added U3: LM1117MP-5.0, Package_TO_SOT_SMD:SOT-223-3_TabPin2, F.Cu at (154.1, 69.1)
