File: pcb/pcb.kicad_sch (KiCad schematic)
At the start: 22 parts, among them J1 USB4085-GF-A_REVB, J2 AudioJack4, J3 AudioJack4, J4 Conn_01x03_Socket, SW1 SW_Push, SW2 SW_Push, SW3 SW_Push, SW4 SW_Push, SW5 SW_Push, SW6 SW_Push, SW7 RotaryEncoder_Switch, SW8 RotaryEncoder_Switch, U1 Pico, U2 Pico, U3 LM1117MP-5.0

Commit message: Changes on MACmini
Parts:
- added J5: Conn_01x03_Socket, symbol Connector:Conn_01x03_Socket
- added J6: Conn_01x08_Pin, symbol Connector:Conn_01x08_Pin
- added R2, R3: 5k1, Capacitor_SMD:C_0603_1608Metric, symbol Device:R
- C1, C2: value C -> 10u; footprint (none) -> Capacitor_SMD:C_0603_1608Metric
- D1, D2, D3, D4: footprint LED_SMD:LED_SK6812MINI_PLCC4_3.5x3.5mm_P1.75mm -> LED_SMD:LED_WS2812B_PLCC4_5.0x5.0mm_P3.2mm
- J2, J3: footprint (none) -> Connector_Audio:Jack_3.5mm_PJ320D_Horizontal
- SW1, SW2, SW3, SW4, SW5, SW6: footprint (none) -> Button_Switch_Keyboard:SW_Cherry_MX_1.00u_PCB
- SW8: footprint (none) -> Rotary_Encoder:RotaryEncoder_Alps_EC11E_Vertical_H20mm
Connections:
- net +5V is gone; now on net VREG_PAD: D1.4 (VDD), D2.4 (VDD), D3.4 (VDD), D4.4 (VDD)
- net VBUS_MAC is gone; now on net VIN_MAC: J3.S
- net GND: now also J1.A1 (GND), J1.A12 (GND), J1.B1 (GND), J1.B12 (GND), R1.1, SW7.C, SW8.C, U2.13 (GND), U2.18 (GND), U2.23 (GND), U2.28 (GND), U2.3 (GND), U2.38 (GND), U2.8 (GND), J6.7 (Pin_7), R2.1, R3.1; no longer R1.2
- net RX_MAC: now also J3.T; no longer J3.R1
- net RX_PAD: now also U2.21 (GPIO16)
- net TX_MAC: now also J3.R1, U2.22 (GPIO17); no longer J3.T
- net VBUS_PAD: no longer C2.1, U3.2 (VO)
- net VIN_MAC: now reaches J1.A4 (VBUS), J1.A9 (VBUS), J1.B4 (VBUS), J1.B9 (VBUS)
- net VIN_MAC: now also U2.40 (VBUS), J6.8 (Pin_8)
- net at J1.A5 (CC1): now also R2.2
- net D+: now reaches J1.A6 (DP1)
- net D+: now also J1.B6 (DP2), U2.45 (TP3)
- net D-: now reaches J1.A7 (DN1)
- net D-: now also J1.B7 (DN2), U2.44 (TP2)
- net at J1.B5 (CC2): now also R3.2
- net at J1.S1 (SHELL), J1.S2 (SHELL), J1.S3 (SHELL)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: now also R1.2
- net Rotary_2A: now reaches SW8.A
- net Rotary_2A: now also U1.16 (GPIO12)
- net Rotary_2B: now reaches SW8.B
- net Rotary_2B: now also U1.17 (GPIO13)
- net DIN: now reaches U2.25 (GPIO19)
- net DIN: now also J6.6 (Pin_6)
- net at U2.41 (SWCLK): now also J5.3 (Pin_3)
- net at U2.42 (GND): now also J5.2 (Pin_2)
- net at U2.43 (SWDIO): now also J5.1 (Pin_1)
- net Rotary_1A: now reaches SW7.A
- net Rotary_1A: now also U1.14 (GPIO10)
- net Rotary_1B: now reaches SW7.B
- net Rotary_1B: now also U1.15 (GPIO11)
- net VREG_PAD: now reaches U1.40 (VBUS)
- net VREG_PAD: now also C2.1, U3.2 (VO)
- no-connect marks 1 -> 21
Other:
- note added: "MAC"
- note added: "PAD"
- note added: "epaper reference: https://www.waveshare.com/1.54inch-e-paper-module.htm"
- note added: "pico reference: https://datasheets.raspberrypi.com/pico/pico-datasheet.pdf"
- moved on the sheet: D1, D2, D3, D4, J1, J2, J3, J4, SW1, SW2, SW3, SW4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

Commit message: Schematic Donezo
Parts:
- J1: footprint USB4085-GF-A_REVB:GCT_USB4085-GF-A_REVB -> USB-C:GCT_USB4085-GF-A_REVB
- J6: footprint (none) -> Connector_PinHeader_2.54mm:PinHeader_1x08_P2.54mm_Vertical
- U1, U2: footprint RPi_Pico:RPi_Pico_SMD_TH -> Library:RPi_Pico_SMD_TH
Connections:
- net DIN: now also U2.5 (GPIO3); no longer U2.25 (GPIO19)
- net RX_MAC: now also U2.21 (GPIO16)
- net RX_PAD: no longer U2.21 (GPIO16)
- net VIN_MAC: no longer J6.8 (Pin_8)
- net BUSY: now reaches J6.1 (Pin_1)
- net BUSY: now also U2.10 (GPIO7)
- net RST: now reaches J6.2 (Pin_2)
- net RST: now also U2.6 (GPIO4)
- net DC: now reaches J6.3 (Pin_3)
- net DC: now also U2.9 (GPIO6)
- net CS: now reaches J6.4 (Pin_4)
- net CS: now also U2.2 (GPIO1)
- net CLK: now reaches J6.5 (Pin_5)
- net CLK: now also U2.4 (GPIO2)
- net 3.3v: now reaches U2.36 (3V3)
- net 3.3v: now also J6.8 (Pin_8)
- no-connect marks 21 -> 44
Changed lines of the file:
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@@
   )
   (no_connect (at 82.55 40.64))
+  (no_connect (at 181.61 110.49))
   (no_connect (at 58.42 33.02))
+  (no_connect (at 181.61 105.41))
+  (no_connect (at 217.17 87.63))
+  (no_connect (at 181.61 107.95))
   (no_connect (at 82.55 66.04))
+  (no_connect (at 217.17 97.79))
+  (no_connect (at 217.17 92.71))
+  (no_connect (at 181.61 102.87))
   (no_connect (at 82.55 60.96))
+  (no_connect (at 217.17 95.25))
+  (no_connect (at 181.61 118.11))
   (no_connect (at 82.55 53.34))
+  (no_connect (at 217.17 107.95))
+  (no_connect (at 181.61 95.25))
+  (no_connect (at 181.61 115.57))
+  (no_connect (at 217.17 72.39))
+  (no_connect (at 181.61 97.79))
   (no_connect (at 82.55 50.8))
   (no_connect (at 72.39 33.02))
+  (no_connect (at 181.61 69.85))
+  (no_connect (at 217.17 82.55))
   (no_connect (at 82.55 45.72))
   (no_connect (at 82.55 63.5))
@@
   (no_connect (at 82.55 71.12))
   (no_connect (at 250.19 109.22))
+  (no_connect (at 217.17 77.47))
   (no_connect (at 82.55 48.26))
+  (no_connect (at 217.17 110.49))
   (no_connect (at 46.99 66.04))
+  (no_connect (at 217.17 102.87))
   (no_connect (at 132.08 156.21))
+  (no_connect (at 217.17 90.17))
+  (no_connect (at 181.61 85.09))
   (no_connect (at 250.19 111.76))
+  (no_connect (at 217.17 85.09))
   (no_connect (at 82.55 78.74))
+  (no_connect (at 217.17 105.41))
   (no_connect (at 46.99 83.82))
   (wire (pts (xy 105.41 114.3) (xy 115.57 114.3))
@@
     (stroke (width 0) (type default))
   )
+  (wire (pts (xy 245.11 64.77) (xy 250.19 64.77))
+    (stroke (width 0) (type default))
+  )
   (wire (pts (xy 92.71 68.58) (xy 82.55 68.58))
     (stroke (width 0) (type default))
@@
     (stroke (width 0) (type default))
   )
+  (wire (pts (xy 177.8 80.01) (xy 181.61 80.01))
+    (stroke (width 0) (type default))
+  )
   (wire (pts (xy 104.14 156.21) (xy 116.84 156.21))
     (stroke (width 0) (type default))
   )
+  (wire (pts (xy 245.11 62.23) (xy 250.19 62.23))
+    (stroke (width 0) (type default))
+  )
   (wire (pts (xy 105.41 127) (xy 115.57 127))
     (stroke (width 0) (type default))
@@
     (stroke (width 0) (type default))
   )
+  (wire (pts (xy 176.53 92.71) (xy 181.61 92.71))
+    (stroke (width 0) (type default))
+  )
   (wire (pts (xy 49.53 116.84) (xy 58.42 116.84))
     (stroke (width 0) (type default))
   )
+  (wire (pts (xy 177.8 72.39) (xy 181.61 72.39))
+    (stroke (width 0) (type default))
+  )
   (wire (pts (xy 50.8 156.21) (xy 62.23 156.21))
     (stroke (width 0) (type default))
@@
     (stroke (width 0) (type default))
   )
+  (wire (pts (xy 177.8 82.55) (xy 181.61 82.55))
+    (stroke (width 0) (type default))
+  )
   (wire (pts (xy 49.53 130.81) (xy 58.42 130.81))
     (stroke (width 0) (type default))
@@
     (stroke (width 0) (type default))
   )
+  (wire (pts (xy 245.11 57.15) (xy 250.19 57.15))
+    (stroke (width 0) (type default))
+  )
   (wire (pts (xy 69.85 116.84) (xy 78.74 116.84))
     (stroke (width 0) (type default))
@@
     (stroke (width 0) (type default))
   )
+  (wire (pts (xy 245.11 49.53) (xy 250.19 49.53))
+    (stroke (width 0) (type default))
+  )
+  (wire (pts (xy 177.8 77.47) (xy 181.61 77.47))
+    (stroke (width 0) (type default))
+  )
   (wire (pts (xy 64.77 92.71) (xy 64.77 91.44))
     (stroke (width 0) (type default))
@@
     (stroke (width 0) (type default))
   )
+  (wire (pts (xy 245.11 67.31) (xy 250.19 67.31))
+    (stroke (width 0) (type default))
+  )
   (wire (pts (xy 36.83 63.5) (xy 46.99 63.5))
     (stroke (width 0) (type default))
   )
+  (wire (pts (xy 245.11 59.69) (xy 250.19 59.69))
+    (stroke (width 0) (type default))
+  )
   (wire (pts (xy 262.89 104.14) (xy 250.19 104.14))
     (stroke (width 0) (type default))
   )
+  (wire (pts (xy 219.71 80.01) (xy 217.17 80.01))
+    (stroke (width 0) (type default))
+  )
   (wire (pts (xy 256.54 114.3) (xy 250.19 114.3))
     (stroke (width 0) (type default))
   )
   (wire (pts (xy 36.83 50.8) (xy 46.99 50.8))
+    (stroke (width 0) (type default))
+  )
+  (wire (pts (xy 177.8 90.17) (xy 181.61 90.17))
     (stroke (width 0) (type default))
   )
@@
     (effects (font (size 1.27 1.27)) (justify left bottom))
   )
+  (label "BUSY" (at 176.53 92.71 0) (fields_autoplaced)
+    (effects (font (size 1.27 1.27)) (justify left bottom))
+  )
   (label "DIN" (at 245.11 54.61 0) (fields_autoplaced)
     (effects (font (size 1.27 1.27)) (justify left bottom))
@@
   )
   (label "Rotary_2B" (at 105.41 132.08 0) (fields_autoplaced)
+    (effects (font (size 1.27 1.27)) (justify left bottom))
+  )
+  (label "DIN" (at 177.8 80.01 0) (fields_autoplaced)
     (effects (font (size 1.27 1.27)) (justify left bottom))
   )
@@
     (effects (font (size 1.27 1.27)) (justify right bottom))
   )
+  (label "RST" (at 245.11 64.77 0) (fields_autoplaced)
+    (effects (font (size 1.27 1.27)) (justify left bottom))
+  )
   (label "VREG_PAD" (at 43.18 148.59 0) (fields_autoplaced)
     (effects (font (size 1.27 1.27)) (justify left bottom))
@@
     (effects (font (size 1.27 1.27)) (justify left bottom))
   )
+  (label "CLK" (at 177.8 77.47 0) (fields_autoplaced)
+    (effects (font (size 1.27 1.27)) (justify left bottom))
+  )
   (label "RX_PAD" (at 82.55 86.36 0) (fields_autoplaced)
     (effects (font (size 1.27 1.27)) (justify left bottom))
@@
     (effects (font (size 1.27 1.27)) (justify left bottom))
   )
+  (label "CS" (at 177.8 72.39 0) (fields_autoplaced)
+    (effects (font (size 1.27 1.27)) (justify left bottom))
+  )
   (label "VREG_PAD" (at 124.46 148.59 0) (fields_autoplaced)
     (effects (font (size 1.27 1.27)) (justify left bottom))
@@
     (effects (font (size 1.27 1.27)) (justify left bottom))
   )
-  (label "RX_PAD" (at 217.17 118.11 0) (fields_autoplaced)
-    (effects (font (size 1.27 1.27)) (justify left bottom))
-  )
-  (label "VIN_MAC" (at 250.19 49.53 180) (fields_autoplaced)
-    (effects (font (size 1.27 1.27)) (justify right bottom))
+  (label "RX_MAC" (at 217.17 118.11 0) (fields_autoplaced)
+    (effects (font (size 1.27 1.27)) (justify left bottom))
   )
   (label "Rotary_1B" (at 36.83 73.66 0) (fields_autoplaced)
@@
     (effects (font (size 1.27 1.27)) (justify left bottom))
   )
-  (label "UART RX->TX Reference: https:{slash}{slash}www.reddit.com{slash}r{slash}raspberrypipico{slash}comments{slash}okb5p9{slash}uart_communication{slash}"
-    (at 13.97 195.58 0) (fields_autoplaced)
-    (effects (font (size 1.27 1.27) (color 194 194 194 1)) (justify left bottom))
-  )
   (label "Rotary_2A" (at 36.83 76.2 0) (fields_autoplaced)
     (effects (font (size 1.27 1.27)) (justify left bottom))
@@
     (effects (font (size 1.27 1.27)) (justify left bottom))
   )
+  (label "3.3v" (at 245.11 49.53 0) (fields_autoplaced)
+    (effects (font (size 1.27 1.27)) (justify left bottom))
+  )
   (label "VIN_MAC" (at 227.33 69.85 180) (fields_autoplaced)
     (effects (font (size 1.27 1.27)) (justify right bottom))
@@
     (effects (font (size 1.27 1.27)) (justify left bottom))
   )
+  (label "3.3v" (at 219.71 80.01 0) (fields_autoplaced)
+    (effects (font (size 1.27 1.27)) (justify left bottom))
+  )
   (label "RX_PAD" (at 119.38 57.15 180) (fields_autoplaced)
     (effects (font (size 1.27 1.27)) (justify right bottom))
   )
-  (label "DIN" (at 217.17 107.95 0) (fields_autoplaced)
-    (effects (font (size 1.27 1.27)) (justify left bottom))
-  )
   (label "LED_SIGNAL" (at 24.13 156.21 0) (fields_autoplaced)
     (effects (font (size 1.27 1.27)) (justify left bottom))
@@
     (effects (font (size 1.27 1.27)) (justify right bottom))
   )
+  (label "RST" (at 177.8 82.55 0) (fields_autoplaced)
+    (effects (font (size 1.27 1.27)) (justify left bottom))
+  )
   (label "TX_PAD" (at 82.55 83.82 0) (fields_autoplaced)
     (effects (font (size 1.27 1.27)) (justify left bottom))
@@
     (effects (font (size 1.27 1.27)) (justify left bottom))
   )
+  (label "BUSY" (at 245.11 67.31 0) (fields_autoplaced)
+    (effects (font (size 1.27 1.27)) (justify left bottom))
+  )
+  (label "CS" (at 245.11 59.69 0) (fields_autoplaced)
+    (effects (font (size 1.27 1.27)) (justify left bottom))
+  )
   (label "Button_6" (at 69.85 130.81 0) (fields_autoplaced)
+    (effects (font (size 1.27 1.27)) (justify left bottom))
+  )
+  (label "DC" (at 245.11 62.23 0) (fields_autoplaced)
     (effects (font (size 1.27 1.27)) (justify left bottom))
   )
@@
   )
   (label "Button_3" (at 69.85 116.84 0) (fields_autoplaced)
+    (effects (font (size 1.27 1.27)) (justify left bottom))
+  )
+  (label "CLK" (at 245.11 57.15 0) (fields_autoplaced)
+    (effects (font (size 1.27 1.27)) (justify left bottom))
+  )
+  (label "DC" (at 177.8 90.17 0) (fields_autoplaced)
     (effects (font (size 1.27 1.27)) (justify left bottom))
   )
@@
       (effects (font (size 1.27 1.27)) (justify right))
     )
-    (property "Footprint" "" (at 255.27 59.69 0)
+    (property "Footprint" "Connector_PinHeader_2.54mm:PinHeader_1x08_P2.54mm_Vertical" (at 255.27 59.69 0)
       (effects (font (size 1.27 1.27)) hide)
     )
@@
       (effects (font (size 1.27 1.27)) (justify left))
     )
-    (property "Footprint" "USB4085-GF-A_REVB:GCT_USB4085-GF-A_REVB" (at 240.03 116.84 0)
+    (property "Footprint" "USB-C:GCT_USB4085-GF-A_REVB" (at 240.03 116.84 0)
       (effects (font (size 1.27 1.27)) (justify bottom) hide)
     )
@@
       (effects (font (size 1.27 1.27)))
     )
-    (property "Footprint" "RPi_Pico:RPi_Pico_SMD_TH" (at 199.39 93.98 90)
+    (property "Footprint" "Library:RPi_Pico_SMD_TH" (at 199.39 93.98 90)
       (effects (font (size 1.27 1.27)) hide)
     )
@@
       (effects (font (size 1.27 1.27)))
     )
-    (property "Footprint" "RPi_Pico:RPi_Pico_SMD_TH" (at 64.77 62.23 90)
-      (effects (font (size 1.27 1.27)) hide)
-    )
+    (property "Footprint" "Library:RPi_Pico_SMD_TH" (at 64.77 62.23 90)
+      (effects (font (size 1.27 1.27)) hide)
+    )
